File: pcb_esp32_wled_pwm_multichannel.kicad_pcb (KiCad board)
At the start: 4 copper layers, 162.6 x 48.3 mm, 105 parts, among them J101 WJ2EDGRC-5.08-4P, J102 WJ2EDGRC-5.08-4P, J103 WJ2EDGRC-5.08-4P, J104 WJ2EDGRC-5.08-4P, J105 Conn_01x05_Male, J106 Conn_01x03_Female, J107 Conn_01x03_Female, J108 Conn_01x02_Female, J109 USB_C_Receptacle_USB2.0, Q101 IRLR8743TRPBF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

Commit message: v3.1 change Cs
Parts:
- removed C108, C109, C110, C115, C118: 100nF/50V, Capacitor_SMD:C_0603_1608Metric
- removed C114: 4.7µF/6.3V(10%), Capacitor_SMD:C_0603_1608Metric
- added C106: CL05A106MQ5NUN, Capacitor_SMD:C_0402_1005Metric, F.Cu at (32.3, 76.5)
- C101: value 220µF/6.3V(20%) -> CL05A106MQ5NUN; footprint Capacitor_SMD:C_1206_3216Metric -> Capacitor_SMD:C_0402_1005Metric
- C102, C105: value 100nF/50V -> CL05A106MQ5NUN; footprint Capacitor_SMD:C_0603_1608Metric -> Capacitor_SMD:C_0402_1005Metric
- C103: value 1µF/50V -> CL05A106MQ5NUN; footprint Capacitor_SMD:C_0603_1608Metric -> Capacitor_SMD:C_0402_1005Metric
- C104: value 10µF/25V -> CL05A106MQ5NUN; footprint Capacitor_SMD:C_0805_2012Metric -> Capacitor_SMD:C_0402_1005Metric
- moved C105 39.2 mm to (31.5, 47.2)
- moved C104 34.2 mm to (25.4, 48.4), turned to 90 degrees
- moved C103 21.2 mm to (12.0, 82.5)
- moved C101 8.93 mm to (11.9, 80.5), turned to 180 degrees
- moved C102 5.30 mm to (12.4, 59.2)
- moved J105 1.53 mm to (14.2, 56.6)
Routing:
- net +3V3: track 74.4 -> 56.9 mm, vias 15 -> 14
- net GND: track 51.2 -> 60.0 mm, vias 74 -> 73
- net /IO0: track 123.1 -> 122.3 mm
