File: pcb_esp32_wled_pwm_multichannel.kicad_sch (KiCad schematic)
At the start: 105 parts, among them J101 WJ2EDGRC-5.08-4P, J102 WJ2EDGRC-5.08-4P, J103 WJ2EDGRC-5.08-4P, J104 WJ2EDGRC-5.08-4P, J105 Conn_01x05_Male, J106 Conn_01x03_Female, J107 Conn_01x03_Female, J108 Conn_01x02_Female, J109 USB_C_Receptacle_USB2.0, Q101 IRLR8743TRPBF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

Commit message: v3.1 change Cs
Parts:
- removed C108, C109, C110, C115, C118: 100nF/50V, Capacitor_SMD:C_0603_1608Metric, symbol Device:C
- removed C114: 4.7µF/6.3V(10%), Capacitor_SMD:C_0603_1608Metric, symbol Device:C
- added C106: CL05A106MQ5NUN, Capacitor_SMD:C_0402_1005Metric, symbol Device:C
- C101: value 220µF/6.3V(20%) -> CL05A106MQ5NUN; footprint Capacitor_SMD:C_1206_3216Metric -> Capacitor_SMD:C_0402_1005Metric; LCSC C412252 -> C15525; MF Murata Electronics -> Samsung Electro-Mechanics; MP GRM31CR60J227ME11L -> CL05A106MQ5NUN
- C102, C105: value 100nF/50V -> CL05A106MQ5NUN; footprint Capacitor_SMD:C_0603_1608Metric -> Capacitor_SMD:C_0402_1005Metric; LCSC C42998 -> C15525; MF FH -> Samsung Electro-Mechanics; MP 0603F104M500NT -> CL05A106MQ5NUN
- C103: value 1µF/50V -> CL05A106MQ5NUN; footprint Capacitor_SMD:C_0603_1608Metric -> Capacitor_SMD:C_0402_1005Metric; LCSC C105174 -> C15525; MF Taiyo Yuden -> Samsung Electro-Mechanics; MP UMK107AB7105KA-T -> CL05A106MQ5NUN
- C104: value 10µF/25V -> CL05A106MQ5NUN; footprint Capacitor_SMD:C_0805_2012Metric -> Capacitor_SMD:C_0402_1005Metric; LCSC C40894 -> C15525; MF FH -> Samsung Electro-Mechanics; MP 0805X106K250NT -> CL05A106MQ5NUN
Connections:
- net +3V3: now also C106.1
- net GND: now also C106.2
Other:
- note added: "C for ESP Espressive recommends 10μF at GND pins in sum. CL05A106MQ5NUN has 3.5μF effC@3.3V so three of those low Z C are perfect and better than 100nFs"
- note removed: "C for ESP"
- moved on the sheet: C101, C112, C113

Commit message: USB-C plug replacement
Parts:
- J109: LCSC C2987386 -> C165948; MF CIKI -> Korean Hroparts Elec; MP TYPE-C-2.0-16PIN-SMT-3 -> TYPE-C-31-M-12
Changed lines of the file:
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@@
 			)
 		)
-		(property "Description" ""
+		(property "Description" "5A 1 16P Female Type-C SMD USB Connectors ROHS"
 			(at 336.55 41.91 0)
 			(effects
@@
 			)
 		)
-		(property "LCSC" "C2987386"
+		(property "LCSC" "C165948"
 			(at 336.55 41.91 0)
 			(effects
@@
 			)
 		)
-		(property "MF" "CIKI"
+		(property "MF" "Korean Hroparts Elec"
 			(at 336.55 41.91 0)
 			(effects
@@
 			)
 		)
-		(property "MP" "TYPE-C-2.0-16PIN-SMT-3"
+		(property "MP" "TYPE-C-31-M-12"
 			(at 336.55 41.91 0)
 			(effects
